File: smart bldc commutator.sch (EAGLE design)
At the start: 41 parts, among them IC1 4011B, Q1 BSS123, Q2 BSS123, Q3 BSS123, Q4 BSS123, Q5 BSS123, Q6 BSS123, Q7 16MHz, U1 ATMEGA328P

Commit message: V3.2 Hardware
One more update
Other:
- note added: "V3.2"
- note removed: "V3.1"
Changed lines of the file:
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@@
 <sheet>
 <plain>
-<text x="184.404" y="17.78" size="2.54" layer="94">V3.1</text>
+<text x="184.404" y="17.78" size="2.54" layer="94">V3.2</text>
 <text x="184.404" y="7.62" size="2.54" layer="94">Nich Fugal</text>
 <text x="99.06" y="144.78" size="5.08" layer="96">A</text>
